Commit message: added gazebo diff drive, inertia needs work

File: goomba_bot/description/robot.urdf.xacro (robot description, xacro)
@@ -1,195 +1,6 @@
-<?xml version="1.0" ?>
-<!-- Generated using onshape-to-robot -->
-<!-- Onshape https://cad.onshape.com/documents/e9064c6d5193bddefb68f171/w/f2e231ecb4ac8838a659f7c8/e/effd3c5c89f281068763c18d -->
-<robot name="goomba_bot">
-  <link name="base_link"></link>
-  <!-- Link base -->
-  <link name="base">
-    <inertial>
-      <origin xyz="0.0929327 -0.0126615 -0.00485732" rpy="0 0 0"/>
-      <mass value="0.208849"/>
-      <inertia ixx="0.000266638" ixy="-5.78139e-07" ixz="-8.08118e-06" iyy="0.000363003" iyz="-1.06903e-07" izz="0.000597738"/>
-    </inertial>
-    <!-- Part base_parts -->
-    <visual>
-      <origin xyz="0.0929327 -0.0126615 -0.00485732" rpy="0 -0 0"/>
-      <geometry>
-        <mesh filename="file:///home/ws/src/goomba_bot/assets/merged/base_visual.stl"/>
-      </geometry>
-      <material name="base_parts_material">
-        <color rgba="0.55 0.55 0.58 1"/>
-      </material>
-    </visual>
-    <collision>
-      <origin xyz="0.0929327 -0.0126615 -0.00485732" rpy="0 -0 0"/>
-      <geometry>
-        <mesh filename="file:///home/ws/src/goomba_bot/assets/merged/base_collision.stl"/>
-      </geometry>
-    </collision>
-  </link>
-  <!-- Link left_wheel -->
-  <link name="left_wheel">
-    <inertial>
-      <origin xyz="-1.8653e-08 1.32e-09 -0.018127" rpy="0 0 0"/>
-      <mass value="0.0296221"/>
-      <inertia ixx="1.19513e-05" ixy="-1e-12" ixz="0" iyy="1.19507e-05" iyz="-0" izz="2.00869e-05"/>
-    </inertial>
-    <!-- Part left_wheel_parts -->
-    <visual>
-      <origin xyz="-1.8653e-08 1.32e-09 -0.018127" rpy="1.5708 -0 -2.55637"/>
-      <geometry>
-        <mesh filename="file:///home/ws/src/goomba_bot/assets/merged/left_wheel_visual.stl"/>
-      </geometry>
-      <material name="left_wheel_parts_material">
-        <color rgba="0.55 0.55 0.58 1"/>
-      </material>
-    </visual>
-    <collision>
-      <origin xyz="-1.8653e-08 1.32e-09 -0.018127" rpy="1.5708 -0 -2.55637"/>
-      <geometry>
-        <mesh filename="file:///home/ws/src/goomba_bot/assets/merged/left_wheel_collision.stl"/>
-      </geometry>
-    </collision>
-  </link>
-  <!-- Joint from base to left_wheel -->
-  <joint name="base_left_wheel" type="continuous">
-    <origin xyz="0.118533 -0.0607433 -0.00814945" rpy="1.5708 0.585227 3.14159"/>
-    <parent link="base"/>
-    <child link="left_wheel"/>
-    <axis xyz="0 0 1"/>
-    <limit effort="10" velocity="10"/>
-  </joint>
-  <!-- Link right_wheel -->
-  <link name="right_wheel">
-    <inertial>
-      <origin xyz="-1.8653e-08 1.32e-09 -0.018127" rpy="0 0 0"/>
-      <mass value="0.0296221"/>
-      <inertia ixx="1.19513e-05" ixy="-1e-12" ixz="0" iyy="1.19507e-05" iyz="-0" izz="2.00869e-05"/>
-    </inertial>
-    <!-- Part right_wheel_parts -->
-    <visual>
-      <origin xyz="-1.8653e-08 1.32e-09 -0.018127" rpy="-1.5708 0 -1.5708"/>
-      <geometry>
-        <mesh filename="file:///home/ws/src/goomba_bot/assets/merged/right_wheel_visual.stl"/>
-      </geometry>
-      <material name="right_wheel_parts_material">
-        <color rgba="0.55 0.55 0.58 1"/>
-      </material>
-    </visual>
-    <collision>
-      <origin xyz="-1.8653e-08 1.32e-09 -0.018127" rpy="-1.5708 0 -1.5708"/>
-      <geometry>
-        <mesh filename="file:///home/ws/src/goomba_bot/assets/merged/right_wheel_collision.stl"/>
-      </geometry>
-    </collision>
-  </link>
-  <!-- Joint from base to right_wheel -->
-  <joint name="base_right_wheel" type="continuous">
-    <origin xyz="0.118569 0.0354816 -0.00814945" rpy="1.5708 -1.5708 0"/>
-    <parent link="base"/>
-    <child link="right_wheel"/>
-    <axis xyz="0 0 1"/>
-    <limit effort="10" velocity="10"/>
-  </joint>
-  <!-- Link lidar -->
-  <link name="lidar">
-    <inertial>
-      <origin xyz="0 0 0" rpy="0 0 0"/>
-      <mass value="1e-09"/>
-      <inertia ixx="1e-09" ixy="0" ixz="0" iyy="1e-09" iyz="0" izz="1e-09"/>
-    </inertial>
-    <!-- Part lidar_parts -->
-    <visual>
-      <origin xyz="-0.157053 -0.0229684 0.0570901" rpy="3.14159 -0 0"/>
-      <geometry>
-        <mesh filename="file:///home/ws/src/goomba_bot/assets/merged/lidar_visual.stl"/>
-      </geometry>
-      <material name="lidar_parts_material">
-        <color rgba="0.55 0.55 0.58 1"/>
-      </material>
-    </visual>
-    <collision>
-      <origin xyz="-0.157053 -0.0229684 0.0570901" rpy="3.14159 -0 0"/>
-      <geometry>
-        <mesh filename="file:///home/ws/src/goomba_bot/assets/merged/lidar_collision.stl"/>
-      </geometry>
-    </collision>
-  </link>
-  <!-- Joint from base to lidar -->
-  <joint name="base_lidar" type="fixed">
-    <origin xyz="0.157053 -0.0229684 0.0570901" rpy="-3.14159 -0 -0"/>
-    <parent link="base"/>
-    <child link="lidar"/>
-    <axis xyz="0 0 1"/>
-    <limit effort="10" velocity="10"/>
-  </joint>
-  <!-- Link imu -->
-  <link name="imu">
-    <inertial>
-      <origin xyz="0 0 0" rpy="0 0 0"/>
-      <mass value="1e-09"/>
-      <inertia ixx="1e-09" ixy="0" ixz="0" iyy="1e-09" iyz="0" izz="1e-09"/>
-    </inertial>
-    <!-- Part imu_parts -->
-    <visual>
-      <origin xyz="-0.080638 -0.00958331 0.0444901" rpy="-3.14159 -0 -0"/>
-      <geometry>
-        <mesh filename="file:///home/ws/src/goomba_bot/assets/merged/imu_visual.stl"/>
-      </geometry>
-      <material name="imu_parts_material">
-        <color rgba="0.55 0.55 0.58 1"/>
-      </material>
-    </visual>
-    <collision>
-      <origin xyz="-0.080638 -0.00958331 0.0444901" rpy="-3.14159 -0 -0"/>
-      <geometry>
-        <mesh filename="file:///home/ws/src/goomba_bot/assets/merged/imu_collision.stl"/>
-      </geometry>
-    </collision>
-  </link>
-  <!-- Joint from base to imu -->
-  <joint name="base_imu" type="fixed">
-    <origin xyz="0.080638 -0.00958331 0.0444901" rpy="3.14159 -0 0"/>
-    <parent link="base"/>
-    <child link="imu"/>
-    <axis xyz="0 0 1"/>
-    <limit effort="10" velocity="10"/>
-  </joint>
-  <!-- Link realsense -->
-  <link name="realsense">
-    <inertial>
-      <origin xyz="0 0 0" rpy="0 0 0"/>
-      <mass value="1e-09"/>
-      <inertia ixx="1e-09" ixy="0" ixz="0" iyy="1e-09" iyz="0" izz="1e-09"/>
-    </inertial>
-    <!-- Part realsense_parts -->
-    <visual>
-      <origin xyz="0.0388416 -0.0363901 0.0136864" rpy="-1.5708 -1.5708 0"/>
-      <geometry>
-        <mesh filename="file:///home/ws/src/goomba_bot/assets/merged/realsense_visual.stl"/>
-      </geometry>
-      <material name="realsense_parts_material">
-        <color rgba="0.55 0.55 0.58 1"/>
-      </material>
-    </visual>
-    <collision>
-      <origin xyz="0.0388416 -0.0363901 0.0136864" rpy="-1.5708 -1.5708 0"/>
-      <geometry>
-        <mesh filename="file:///home/ws/src/goomba_bot/assets/merged/realsense_collision.stl"/>
-      </geometry>
-    </collision>
-  </link>
-  <!-- Joint from base to realsense -->
-  <joint name="base_realsense" type="fixed">
-    <origin xyz="-0.0136864 -0.0388416 0.0363901" rpy="1.5708 0 1.5708"/>
-    <parent link="base"/>
-    <child link="realsense"/>
-    <axis xyz="0 0 1"/>
-    <limit effort="10" velocity="10"/>
-  </joint>
-  <joint name="base_link_base" type="fixed">
-    <origin xyz="0 0 0" rpy="0 0 0"/>
-    <parent link="base_link"/>
-    <child link="base"/>
-  </joint>
+<?xml version="1.0"?>
+<robot xmlns:xacro="http://www.ros.org/wiki/xacro"  name="robot">
+    <xacro:include filename="inertial.xacro" />
+    <xacro:include filename="robot_core.xacro" />
+    <xacro:include filename="gazebo_control.xacro" />
 </robot>
