Commit message: removing joint limits, added data collector node, added script for 'default' test route on map

File: goomba_bot/description/lidar.xacro (robot description, xacro)
@@ -10,5 +10,5 @@
                 <scan>
                     <horizontal>
-                        <samples>360</samples>
+                        <samples>128</samples>
                         <min_angle>-3.14</min_angle>
                         <max_angle>3.14</max_angle>

File: goomba_bot/description/robot_core.xacro (robot description, xacro)
@@ -67,5 +67,4 @@
     <child link="left_wheel"/>
     <axis xyz="0 0 1"/>
-    <limit effort="10" velocity="10"/>
   </joint>
   <!-- Link right_wheel -->
@@ -99,5 +98,4 @@
     <child link="right_wheel"/>
     <axis xyz="0 0 1"/>
-    <limit effort="10" velocity="10"/>
   </joint>
   <!-- Link lidar -->
@@ -131,5 +129,4 @@
     <child link="lidar"/>
     <axis xyz="0 0 1"/>
-    <limit effort="10" velocity="10"/>
   </joint>
   <!-- Link imu -->
@@ -163,5 +160,4 @@
     <child link="imu"/>
     <axis xyz="0 0 1"/>
-    <limit effort="10" velocity="10"/>
   </joint>
   <!-- Link realsense -->
@@ -195,5 +191,4 @@
     <child link="realsense"/>
     <axis xyz="0 0 1"/>
-    <limit effort="10" velocity="10"/>
   </joint>
   <!-- Link caster_wheel -->
